File: GameBoyCartridgeBreakout.kicad_pcb (KiCad board)
At the start: 2 copper layers, 51 x 61 mm, 2 parts, among them J1 Conn_02x16_Odd_Even, U1 GAMEBOY_CART_EDGE

Commit message: Generate gerbers
Other:
- board text added: "GAME BOY CARTRIDGE BREAKOUT v1.0"
- board text added: "JWG 2019-09-21"
Changed lines of the file:
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@@
   (general
     (thickness 1.6)
-    (drawings 12)
+    (drawings 14)
     (tracks 165)
     (zones 0)
@@
     (47 F.CrtYd user)
     (48 B.Fab user)
-    (49 F.Fab user)
+    (49 F.Fab user hide)
   )
   (setup
@@
     (visible_elements 7FFFF7FF)
     (pcbplotparams
-      (layerselection 0x010fc_ffffffff)
-      (usegerberextensions false)
+      (layerselection 0x010f0_ffffffff)
+      (usegerberextensions true)
       (usegerberattributes false)
       (usegerberadvancedattributes false)
@@
       (psnegative false)
       (psa4output false)
-      (plotreference true)
+      (plotreference false)
       (plotvalue true)
       (plotinvisibletext false)
@@
       (outputformat 1)
       (mirror false)
-      (drillshape 1)
+      (drillshape 0)
       (scaleselection 1)
-      (outputdirectory ""))
+      (outputdirectory "gerbers"))
   )
   (net 0 "")
@@
     (at 150 100)
     (attr smd)
-    (fp_text reference U1 (at 0 4.5) (layer F.SilkS)
+    (fp_text reference U1 (at 0 4.5) (layer F.SilkS) hide
       (effects (font (size 1 1) (thickness 0.15)))
     )
@@
     )
   )
+  (gr_text "JWG 2019-09-21" (at 128.4 43.5) (layer B.SilkS)
+    (effects (font (size 0.5 0.5) (thickness 0.1)) (justify mirror))
+  )
+  (gr_text "GAME BOY CARTRIDGE BREAKOUT v1.0" (at 150 57.9) (layer F.SilkS)
+    (effects (font (size 1.5 1.5) (thickness 0.3)))
+  )
   (gr_circle (center 150 88.25) (end 153.5 88.25) (layer Edge.Cuts) (width 0.05))
